Commit message: 08804_GPUrent_sync

File: src/cobot_rg2/onrobot-ros2/onrobot_rg_description/urdf/onrobot_rg2_model_macro.xacro (robot description, xacro)
@@ -132,7 +132,7 @@
   </xacro:macro>
   <xacro:macro name="right_outer_knuckle_joint" params="prefix">
-    <joint name="${prefix}base_link" type="revolute">
+    <joint name="${prefix}right_outer_knuckle_joint" type="revolute">
       <origin xyz="0 0.017178 0.125797" rpy="0 0 ${pi}" />
-      <parent link="${prefix}onrobot_rg2_base_link" />
+      <parent link="${prefix}base_link" />
       <child link="${prefix}right_outer_knuckle" />
       <axis xyz="1 0 0" />
